Commit message: Add SCARA robot workspace table, conveyor track, pick-and-place automation, teleop scripts, and MuJoCo simulation support

File: urdf/arm.xacro (robot description, xacro)
@@ -1,6 +1,8 @@
 <?xml version="1.0" ?>
 <robot name="scara" xmlns:xacro="http://www.ros.org/wiki/xacro">
-    <link name="world"/>
     <!-- Materials -->
+    <material name="scara_wood_brown">
+        <color rgba="0.75 0.52 0.32 1.0"/>
+    </material>
     <material name="scara_mid_blue">
         <color rgba="0.0 0.4 0.8 1.0"/>
@@ -12,4 +14,31 @@
         <color rgba="0.7 0.7 0.7 1.0"/>
     </material>
+    <!-- ── WOODEN TABLE BASE PLATFORM ────────────────────────────── -->
+    <link name="table_link">
+        <visual>
+            <origin xyz="0.25 0 -0.10" rpy="0 0 0"/>
+            <geometry>
+                <box size="1.20 0.85 0.20"/>
+            </geometry>
+            <material name="scara_wood_brown"/>
+        </visual>
+        <collision>
+            <origin xyz="0.25 0 -0.10" rpy="0 0 0"/>
+            <geometry>
+                <box size="1.20 0.85 0.20"/>
+            </geometry>
+        </collision>
+        <inertial>
+            <origin xyz="0.25 0 -0.10" rpy="0 0 0"/>
+            <mass value="50.0"/>
+            <inertia ixx="1.0" ixy="0.0" ixz="0.0" iyy="1.0" iyz="0.0" izz="1.0"/>
+        </inertial>
+    </link>
+    <!-- Joint mounting SCARA robot base on top of the wooden table -->
+    <joint name="table_to_base_joint" type="fixed">
+        <origin xyz="0.05 0.08 0.0" rpy="0 0 0"/>
+        <parent link="table_link"/>
+        <child link="base_link"/>
+    </joint>
     <!-- ── BASE ─────────────────────────────────────── -->
     <link name="base_link">
@@ -37,9 +66,4 @@
         </inertial>
     </link>
-    <joint name="base_joint" type="fixed">
-        <origin xyz="0 0 0" rpy="0 0 0"/>
-        <parent link="world"/>
-        <child link="base_link"/>
-    </joint>
     <!-- ── COLUMN ────────────────────────────────────── -->
     <link name="column_link">
@@ -247,5 +271,5 @@
     <link name="right_finger_joint_mimic_dummy"/>
     <joint name="right_finger_joint_mimic" type="fixed">
-        <parent link="world"/>
+        <parent link="base_link"/>
         <child link="right_finger_joint_mimic_dummy"/>
     </joint>
@@ -281,4 +305,7 @@
         </joint>
     </ros2_control>
+    <gazebo reference="table_link">
+        <material>Gazebo/Wood</material>
+    </gazebo>
     <gazebo>
         <plugin filename="ign_ros2_control-system" name="ign_ros2_control::IgnitionROS2ControlPlugin">

Commit message: Fix Gazebo SCARA alignment and joystick gripper

File: urdf/arm.xacro (robot description, xacro)
@@ -101,5 +101,5 @@
     <link name="shoulder_link">
         <visual>
-            <origin xyz="-0.045 0 -0.39" rpy="0 0 0"/>
+            <origin xyz="-0.059954333 -0.059974857 -0.390000" rpy="0 0 0"/>
             <geometry>
                 <mesh filename="package://scara_description/meshes/shoulder_link.stl"
@@ -109,5 +109,5 @@
         </visual>
         <collision>
-            <origin xyz="-0.045 0 -0.39" rpy="0 0 0"/>
+            <origin xyz="-0.059954333 -0.59974857 -0.390000" rpy="0 0 0"/>
             <geometry>
                 <mesh filename="package://scara_description/meshes/shoulder_link.stl"
@@ -266,5 +266,4 @@
         <axis xyz="0 -1 0"/>
         <limit lower="-0.06" upper="0.0" effort="100.0" velocity="0.5"/>
-        <mimic joint="left_finger_joint" multiplier="1.0" offset="0.0"/>
     </joint>
     <!-- DUMMY JOINT FOR MOVEIT2-->
@@ -304,4 +303,9 @@
             <state_interface name="velocity"/>
         </joint>
+        <joint name="right_finger_joint">
+    <command_interface name="position"/>
+    <state_interface name="position"/>
+    <state_interface name="velocity"/>
+</joint>
     </ros2_control>
     <gazebo reference="table_link">
@@ -309,7 +313,8 @@
     </gazebo>
     <gazebo>
-        <plugin filename="ign_ros2_control-system" name="ign_ros2_control::IgnitionROS2ControlPlugin">
-            <parameters>$(find scara_description)/config/scara_controllers.yaml</parameters>
-        </plugin>
-    </gazebo>
+    <plugin filename="gz_ros2_control-system"
+            name="gz_ros2_control::GazeboSimROS2ControlPlugin">
+        <parameters>$(find scara_description)/config/scara_controllers.yaml</parameters>
+    </plugin>
+</gazebo>
 </robot>
